Commit message: 02/10/2568#1

File: src/hexapod_description/robot/visual/gazebo_full.xacro (robot description, xacro)
@@ -5,4 +5,15 @@
       <plugin>gz_ros2_control/GazeboSimSystem</plugin>
     </hardware>
+    <joint name="rail_to_slider">
+      <command_interface name="effort">
+        <param name="min">-1000</param>
+        <param name="max">1000</param>
+      </command_interface>
+      <state_interface name="position">
+        <param name="initial_value">0.0</param>
+      </state_interface>
+      <state_interface name="velocity"/>
+      <state_interface name="effort"/>
+    </joint>
     <joint name="base_joint">
       <command_interface name="effort">

File: src/hexapod_description/robot/visual/hexapod.xacro (robot description, xacro)
@@ -3,20 +3,93 @@
     <xacro:include filename="inertial_macros.xacro" />
     <xacro:include filename="hexapod_params.xacro" />
-    <xacro:include filename="robot_material.xacro" />\
+    <xacro:include filename="robot_material.xacro" />
     <xacro:include filename="gazebo_full.xacro" />
-    <!-- BASE LINK -->
-    <link name="world"/>
-    <joint name="world_to_base" type="fixed">
+    <!-- WORLD LINK -->
+    <link name="world">
+        <inertial>
+            <mass value="0.001"/>
+            <inertia ixx="0.000001" ixy="0" ixz="0" iyy="0.000001" iyz="0" izz="0.000001"/>
+        </inertial>
+    </link>
+    <!-- LINEAR GUIDE BOX (RAIL) -->
+    <joint name="world_to_rail" type="fixed">
         <parent link="world"/>
+        <child link="linear_rail"/>
+        <origin xyz="0 0 ${world_height}" rpy="0 0 0"/>
+    </joint>
+    <link name="linear_rail">
+        <inertial>
+            <origin xyz="0 0 0" rpy="0 0 0" />
+            <mass value="1.0" />
+            <inertia
+                ixx="0.01"
+                ixy="0"
+                ixz="0"
+                iyy="0.01"
+                iyz="0"
+                izz="0.001" />
+        </inertial>
+        <visual>
+            <origin xyz="0 0 0" rpy="0 0 0" />
+            <geometry>
+                <!-- Rail dimensions: length=4m, width=0.1m, height=0.05m -->
+                <box size="0.1 4.0 0.05"/>
+            </geometry>
+            <material name="grey">
+                <color rgba="0.5 0.5 0.5 1.0"/>
+            </material>
+        </visual>
+        <collision>
+            <origin xyz="0 0 0" rpy="0 0 0" />
+            <geometry>
+                <box size="0.1 4.0 0.05"/>
+            </geometry>
+        </collision>
+    </link>
+    <!-- SLIDER THAT MOVES ALONG THE RAIL -->
+    <joint name="rail_to_slider" type="prismatic">
+        <parent link="linear_rail"/>
+        <child link="slider"/>
+        <origin xyz="0 0 0.05" rpy="0 0 0"/>
+        <axis xyz="0 1 0"/>  <!-- Moves along Y-axis (along the rail) -->
+        <limit effort="1000" velocity="10" lower="-1.8" upper="1.8"/>
+        <dynamics damping="10.0" friction="1.0"/>
+    </joint>
+    <link name="slider">
+        <inertial>
+            <origin xyz="0 0 0" rpy="0 0 0" />
+            <mass value="0.1" />
+            <inertia
+                ixx="0.0001"
+                ixy="0"
+                ixz="0"
+                iyy="0.0001"
+                iyz="0"
+                izz="0.0001" />
+        </inertial>
+        <visual>
+            <origin xyz="0 0 0" rpy="0 0 0" />
+            <geometry>
+                <!-- Slider dimensions: smaller box that rides on the rail -->
+                <box size="0.08 0.08 0.03"/>
+            </geometry>
+            <material name="blue">
+                <color rgba="0.2 0.2 0.8 1.0"/>
+            </material>
+        </visual>
+        <collision>
+            <origin xyz="0 0 0" rpy="0 0 0" />
+            <geometry>
+                <box size="0.08 0.08 0.03"/>
+            </geometry>
+        </collision>
+    </link>
+    <!-- CONNECT SLIDER TO BASE_LINK -->
+    <joint name="slider_to_base" type="fixed">
+        <parent link="slider"/>
         <child link="base_link"/>
-        <origin xyz="0 0 ${world_height}" rpy="0 0 0"/>
-    </joint>
-    <!-- <joint name="world_to_base" type="prismatic">
-        <parent link="world"/>
-        <child link="base_link"/>
-        <origin xyz="0 0 ${world_height}" rpy="0 0 0"/>
-        <axis xyz="0 1 0"/>
-        <limit effort="1000" velocity="10" lower="-2" upper="2"/>
-    </joint> -->
+        <origin xyz="0 0 0.02" rpy="0 0 0"/>
+    </joint>
+    <!-- HEXAPOD LEG STARTS HERE -->
     <link name="base_link">
         <inertial>
