Commit message: 002

File: src/system_identification_description/robot/visual/hip_link_only.xacro (robot description, xacro)
@@ -75,5 +75,5 @@
             <origin xyz="0 0 0" rpy="0 0 0" />
             <geometry>
-                <mesh filename="package://test_station_description/meshes/hip_link_v2.STL" />
+                <mesh filename="package://system_identification_description/meshes/hip_link_v2.STL" />
             </geometry>
             <material name="green" />
@@ -83,5 +83,5 @@
             <origin xyz="0 0 0" rpy="0 0 0" />
             <geometry>
-                <mesh filename="package://test_station_description/meshes/hip_link_v2.STL" />
+                <mesh filename="package://system_identification_description/meshes/hip_link_v2.STL" />
             </geometry>
         </collision>

Commit message: ReadME

File: src/system_identification_description/robot/visual/hip_link_only.xacro (robot description, xacro)
@@ -34,5 +34,5 @@
     <xacro:property name="hip_iyy" value="0.00120" />
     <xacro:property name="hip_iyz" value="0.0" />
-    <xacro:property name="hip_izz" value="0.00050" />
+    <xacro:property name="hip_izz" value="0.0005" />
     <!-- ====================================================================== -->
     <!-- WORLD LINK (Fixed Root)                                                -->
@@ -54,5 +54,5 @@
         <axis xyz="0 0 1" />
         <!-- No damping or friction for free pendulum motion -->
-        <dynamics damping="0.00040" friction="0.00280" />
+        <dynamics damping="0.000325" friction="0.00270" />
     </joint>
     <!-- ====================================================================== -->
