Commit message: compare

File: src/system_identification_description/robot/visual/ankle_link_only.xacro (robot description, xacro)
@@ -56,8 +56,8 @@
         <parent link="world" />
         <child link="ankle_link" />
-        <!-- Position: 1.0m above ground -->
-        <origin xyz="0 0 1.0" rpy="0 0 0" />
+        <!-- Position: 1.0 m above ground -->
+        <origin xyz="0 0 0.3" rpy="0 1.5701 0" />
         <!-- Rotation axis: Y-axis (pitch motion) -->
-        <axis xyz="0 1 0" />
+        <axis xyz="0 0 1" />
         <!-- Joint limits -->
         <limit effort="${joint_effort_limit}" velocity="${joint_velocity_limit}" />

File: src/system_identification_description/robot/visual/hip_link_gazebo.xacro (robot description, xacro)
@@ -13,5 +13,5 @@
     <!-- ====================================================================== -->
     <xacro:arg name="controller_config_file"
-               default="$(find test_station_simulation)/config/hip_pendulum_controller.yaml" />
+               default="$(find system_identification_simulation)/config/hip_pendulum_controller.yaml" />
     <!-- ====================================================================== -->
     <!-- ROS2 CONTROL SYSTEM                                                    -->

File: src/system_identification_description/robot/visual/hip_link_only.xacro (robot description, xacro)
@@ -34,5 +34,5 @@
     <xacro:property name="hip_iyy" value="0.00120" />
     <xacro:property name="hip_iyz" value="0.0" />
-    <xacro:property name="hip_izz" value="0.0005" />
+    <xacro:property name="hip_izz" value="0.000425" />
     <!-- ====================================================================== -->
     <!-- WORLD LINK (Fixed Root)                                                -->
@@ -54,5 +54,5 @@
         <axis xyz="0 0 1" />
         <!-- No damping or friction for free pendulum motion -->
-        <dynamics damping="0.000325" friction="0.00270" />
+        <dynamics damping="0.000375" friction="0.00350" />
     </joint>
     <!-- ====================================================================== -->

File: src/system_identification_description/robot/visual/knee_link_gazebo.xacro (robot description, xacro)
@@ -13,5 +13,5 @@
     <!-- ====================================================================== -->
     <xacro:arg name="controller_config_file"
-               default="$(find test_station_simulation)/config/knee_pendulum_controller.yaml" />
+               default="$(find system_identification_simulation)/config/knee_pendulum_controller.yaml" />
     <!-- ====================================================================== -->
     <!-- ROS2 CONTROL SYSTEM                                                    -->
@@ -31,5 +31,5 @@
             <!-- State Interfaces: Position, Velocity, Effort -->
             <state_interface name="position">
-                <param name="initial_value"> 0.0 </param>
+                <param name="initial_value"> -0.78539 </param>
             </state_interface>
             <state_interface name="velocity" />

File: src/system_identification_description/robot/visual/knee_link_only.xacro (robot description, xacro)
@@ -81,5 +81,5 @@
             <origin xyz="0 0 0" rpy="0 0 0" />
             <geometry>
-                <mesh filename="package://test_station_description/meshes/knee_link_v2.STL" />
+                <mesh filename="package://system_identification_description/meshes/knee_link_v2.STL" />
             </geometry>
             <material name="blue" />
@@ -89,5 +89,5 @@
             <origin xyz="0 0 0" rpy="0 0 0" />
             <geometry>
-                <mesh filename="package://test_station_description/meshes/knee_link_v2.STL" />
+                <mesh filename="package://system_identification_description/meshes/knee_link_v2.STL" />
             </geometry>
         </collision>
